Commit message: Fix the vertical offset of the model

File: urdf/flir_a400.urdf.xacro (robot description, xacro)
@@ -10,5 +10,5 @@
           <color rgba="0 0 0 1" />
         </material>
-        <origin xyz="0 0 0" rpy="1.5707963267948966 0 1.5707963267948966" />
+        <origin xyz="0 0 0.038 " rpy="1.5707963267948966 0 1.5707963267948966" />
       </visual>
       <collision>
@@ -16,5 +16,5 @@
           <mesh filename="package://camera_aravis/meshes/flir_a400.stl" scale="0.001 0.001 0.001" />
         </geometry>
-        <origin xyz="0 0 0" rpy="1.5707963267948966 0 1.5707963267948966" />
+        <origin xyz="0 0 0.038" rpy="1.5707963267948966 0 1.5707963267948966" />
       </collision>
     </link>
@@ -25,3 +25,6 @@
     </joint>
   </xacro:macro>
+  <xacro:flir_a400 prefix="a400" parent_link="front_mount">
+    <origin xyz="0 0 0" rpy="0 0 0" />
+  </xacro:flir_a400>
 </robot>

Commit message: Remove the testing stub

File: urdf/flir_a400.urdf.xacro (robot description, xacro)
@@ -25,6 +25,3 @@
     </joint>
   </xacro:macro>
-  <xacro:flir_a400 prefix="a400" parent_link="front_mount">
-    <origin xyz="0 0 0" rpy="0 0 0" />
-  </xacro:flir_a400>
 </robot>
