Commit message: Separate the driver from the description

File: camera_aravis_description/urdf/flir_a400.urdf.xacro (robot description, xacro)
@@ -5,5 +5,5 @@
       <visual>
         <geometry>
-          <mesh filename="package://camera_aravis/meshes/flir_a400.stl" scale="0.001 0.001 0.001" />
+          <mesh filename="package://camera_aravis_description/meshes/flir_a400.stl" scale="0.001 0.001 0.001" />
         </geometry>
         <material name="black">

Commit message: Fixed path to collision mesh

File: camera_aravis_description/urdf/flir_a400.urdf.xacro (robot description, xacro)
@@ -14,5 +14,5 @@
       <collision>
         <geometry>
-          <mesh filename="package://camera_aravis/meshes/flir_a400.stl" scale="0.001 0.001 0.001" />
+          <mesh filename="package://camera_aravis_description/meshes/flir_a400.stl" scale="0.001 0.001 0.001" />
         </geometry>
         <origin xyz="0 0 0.038" rpy="1.5707963267948966 0 1.5707963267948966" />
